Commit message: Created robot description with diff_drive and imu

File: src/micromouse_description/urdf/micromouse_description.xacro (robot description, xacro)
@@ -1,4 +1,5 @@
 <?xml version="1.0"?>
-<robot name="micromouse" xmlns:xacro="http://ros.org/wiki/xacro">
+<robot name="sam_bot" xmlns:xacro="http://ros.org/wiki/xacro">
+    <xacro:include filename="$(find micromouse_description)/urdf/macros.xacro" />
     <!-- Define robot constants -->
     <xacro:property name="base_width" value="0.09" />
@@ -7,5 +8,5 @@
     <xacro:property name="wheel_radius" value="0.02" />
     <xacro:property name="wheel_width" value="0.01" />
-    <xacro:property name="wheel_ygap" value="0.0025" />
+    <xacro:property name="wheel_ygap" value="${base_width/2 + wheel_width/2}" />
     <xacro:property name="wheel_zoff" value="0.005" />
     <xacro:property name="wheel_xoff" value="0.02" />
@@ -15,13 +16,21 @@
         <visual>
             <geometry>
-                <cylinder radius="${base_width/2}" length="${base_height}" />
+                <cylinder radius="${base_width}" length="${base_height}" />
             </geometry>
-            <material name="Green">
-                <color rgba="0 1.0 0.6 1.0" />
+            <material name="Cyan">
+                <color rgba="0 1.0 1.0 1.0" />
             </material>
         </visual>
+        <collision>
+            <geometry>
+                <cylinder radius="${base_width}" length="${base_height}" />
+            </geometry>
+        </collision>
+        <xacro:box_inertia m="15" w="${base_width}" d="${base_length}" h="${base_height}" />
     </link>
     <!-- Robot Footprint -->
-    <link name="base_footprint" />
+    <link name="base_footprint">
+        <xacro:box_inertia m="0" w="0" d="0" h="0" />
+    </link>
     <joint name="base_joint" type="fixed">
         <parent link="base_link" />
@@ -41,6 +50,13 @@
                 </material>
             </visual>
+            <collision>
+                <origin xyz="0 0 0" rpy="${pi/2} 0 0" />
+                <geometry>
+                    <cylinder radius="${wheel_radius}" length="${wheel_width}" />
+                </geometry>
+            </collision>
+            <xacro:cylinder_inertia m="0.5" r="${wheel_radius}" h="${wheel_width}" />
         </link>
-        <joint name="${prefix}_joint" type="fixed">
+        <joint name="${prefix}_joint" type="continuous">
             <parent link="base_link" />
             <child link="${prefix}_link" />
@@ -51,5 +67,4 @@
     <xacro:wheel prefix="drivewhl_l" x_reflect="-1" y_reflect="1" />
     <xacro:wheel prefix="drivewhl_r" x_reflect="-1" y_reflect="-1" />
-    <!-- Caster Wheel -->
     <link name="front_caster">
         <visual>
@@ -61,4 +76,11 @@
             </material>
         </visual>
+        <collision>
+            <origin xyz="0 0 0" rpy="0 0 0" />
+            <geometry>
+                <sphere radius="${(wheel_radius+wheel_zoff-(base_height/2))}" />
+            </geometry>
+        </collision>
+        <xacro:sphere_inertia m="0.5" r="${(wheel_radius+wheel_zoff-(base_height/2))}" />
     </link>
     <joint name="caster_joint" type="fixed">
@@ -67,3 +89,5 @@
         <origin xyz="${caster_xoff} 0.0 ${-(base_height/2)}" rpy="0 0 0" />
     </joint>
+    <xacro:include filename="$(find micromouse_description)/urdf/imu.xacro" />
+    <xacro:include filename="$(find micromouse_description)/urdf/diff_drive.xacro" />
 </robot>

Commit message: Added distance sensors

File: src/micromouse_description/urdf/micromouse_description.xacro (robot description, xacro)
@@ -91,3 +91,15 @@
     <xacro:include filename="$(find micromouse_description)/urdf/imu.xacro" />
     <xacro:include filename="$(find micromouse_description)/urdf/diff_drive.xacro" />
+    <!-- Range Sensors -->
+    <xacro:include filename="$(find micromouse_description)/urdf/range_sensor.xacro" />
+    <xacro:range_sensor name="range_sesnor_right" parent="base_link">
+        <origin xyz="0.05 0.05 ${base_height/2 + 0.005}" rpy="0 0 -${3.14/6}" />
+    </xacro:range_sensor>
+    <xacro:range_sensor name="range_sensor_left" parent="base_link">
+        <origin xyz="0.05 -0.05 ${base_height/2 + 0.005}" rpy="0 0 ${3.14/6}" />
+    </xacro:range_sensor>
+<!--
+    <xacro:range_sensor name="range_sensor_front" parent="base_link">
+        <origin xyz="0.05 0.0 ${base_height/2 + 0.005}" rpy="0 0 0" />
+    </xacro:range_sensor> -->
 </robot>
