Commit message: managed sensors

File: ws/src/micromouse_description/urdf/range_sensor.xacro (robot description, xacro)
@@ -12,13 +12,4 @@
                 </material>
             </visual>
-            <collision>
-                <origin rpy="0 0 0" xyz="0 0 0" />
-                <geometry>
-                    <cylinder length="0.01" radius="0.01" />
-                </geometry>
-                <material name="Black">
-                    <color rgba="0.0 0.0 0.0 1.0" />
-                </material>
-            </collision>
         </link>
         <joint name="${name}_joint" type="fixed">
@@ -35,12 +26,19 @@
                         <horizontal>
                             <samples>10</samples>
-                            <resolution>1.0</resolution>
-                            <min_angle>-0.1</min_angle>
-                            <max_angle>0.1</max_angle>
+                            <resolution>1</resolution>
+                            <min_angle>-0.05</min_angle>
+                            <max_angle>0.05</max_angle>
                         </horizontal>
+                        <vertical>
+                            <samples>10</samples>
+                            <resolution>1</resolution>
+                            <min_angle>-0.05</min_angle>
+                            <max_angle>0.05</max_angle>
+                        </vertical>
                     </scan>
                     <range>
                         <min>0.01</min>
                         <max>0.5</max>
+                        <resolution>0.01</resolution>
                     </range>
                 </ray>
