Commit message: Added colours to robot

File: ws/src/micromouse_description/urdf/diff_drive.xacro (robot description, xacro)
@@ -23,3 +23,9 @@
         </plugin>
     </gazebo>
+    <gazebo reference="drivewhl_l_link">
+        <material>Gazebo/Black</material>
+    </gazebo>
+    <gazebo reference="drivewhl_r_link">
+        <material>Gazebo/Black</material>
+    </gazebo>
 </robot>

File: ws/src/micromouse_description/urdf/imu.xacro (robot description, xacro)
@@ -20,4 +20,5 @@
 </joint>
 <gazebo reference="imu_link">
+    <material>Gazebo/Black</material>
     <sensor name="imu_sensor" type="imu">
         <plugin filename="libgazebo_ros_imu_sensor.so" name="imu_plugin">

File: ws/src/micromouse_description/urdf/micromouse_description.xacro (robot description, xacro)
@@ -29,4 +29,7 @@
         <xacro:box_inertia m="15" w="${base_width}" d="${base_length}" h="${base_height}" />
     </link>
+    <gazebo reference="base_link">
+        <material>Gazebo/Turquoise</material>
+    </gazebo>
     <!-- Robot Footprint -->
     <link name="base_footprint">
@@ -89,4 +92,7 @@
         <origin xyz="${caster_xoff} 0.0 ${-(base_height/2)}" rpy="0 0 0" />
     </joint>
+    <gazebo reference="front_caster">
+        <material>Gazebo/Black</material>
+    </gazebo>
     <xacro:include filename="$(find micromouse_description)/urdf/imu.xacro" />
     <xacro:include filename="$(find micromouse_description)/urdf/diff_drive.xacro" />
