Commit message: setup the world

File: ws/src/micromouse_description/urdf/micromouse_description.xacro (robot description, xacro)
@@ -3,6 +3,6 @@
     <xacro:include filename="$(find micromouse_description)/urdf/macros.xacro" />
     <!-- Define robot constants -->
-    <xacro:property name="base_width" value="0.09" />
-    <xacro:property name="base_length" value="0.1" />
+    <xacro:property name="base_width" value="0.04" />
+    <xacro:property name="base_length" value="0.06" />
     <xacro:property name="base_height" value="0.025" />
     <xacro:property name="wheel_radius" value="0.02" />
@@ -10,5 +10,5 @@
     <xacro:property name="wheel_ygap" value="${base_width/2 + wheel_width/2}" />
     <xacro:property name="wheel_zoff" value="0.005" />
-    <xacro:property name="wheel_xoff" value="0.02" />
+    <xacro:property name="wheel_xoff" value="0.015" />
     <xacro:property name="caster_xoff" value="0.04" />
     <!-- Robot Base -->
@@ -100,11 +100,11 @@
     <xacro:include filename="$(find micromouse_description)/urdf/range_sensor.xacro" />
     <xacro:range_sensor name="range_sensor_right" parent="base_link">
-        <origin xyz="0.05 0.05 ${base_height/2 + 0.005}" rpy="0 0 -${3.14/6}" />
+        <origin xyz="0.025 0.025 ${base_height/2 + 0.005}" rpy="0 0 -${3.14/6}" />
     </xacro:range_sensor>
     <xacro:range_sensor name="range_sensor_left" parent="base_link">
-        <origin xyz="0.05 -0.05 ${base_height/2 + 0.005}" rpy="0 0 ${3.14/6}" />
+        <origin xyz="0.025 -0.025 ${base_height/2 + 0.005}" rpy="0 0 ${3.14/6}" />
     </xacro:range_sensor>
     <xacro:range_sensor name="range_sensor_front" parent="base_link">
-        <origin xyz="0.05 0.0 ${base_height/2 + 0.005}" rpy="0 0 0" />
+        <origin xyz="0.025 0.0 ${base_height/2 + 0.005}" rpy="0 0 0" />
     </xacro:range_sensor>
 </robot>

File: ws/src/micromouse_description/urdf/range_sensor.xacro (robot description, xacro)
@@ -6,5 +6,5 @@
                 <origin rpy="0 0 0" xyz="0 0 0" />
                 <geometry>
-                    <cylinder length="0.01" radius="0.01" />
+                    <cylinder length="0.005" radius="0.005" />
                 </geometry>
                 <material name="Black">

Commit message: Added PID controller to center tunnel driving

File: ws/src/micromouse_description/urdf/micromouse_description.xacro (robot description, xacro)
@@ -3,6 +3,6 @@
     <xacro:include filename="$(find micromouse_description)/urdf/macros.xacro" />
     <!-- Define robot constants -->
-    <xacro:property name="base_width" value="0.04" />
-    <xacro:property name="base_length" value="0.06" />
+    <xacro:property name="base_width" value="0.035" />
+    <xacro:property name="base_length" value="0.05" />
     <xacro:property name="base_height" value="0.025" />
     <xacro:property name="wheel_radius" value="0.02" />
@@ -100,11 +100,14 @@
     <xacro:include filename="$(find micromouse_description)/urdf/range_sensor.xacro" />
     <xacro:range_sensor name="range_sensor_right" parent="base_link">
-        <origin xyz="0.025 0.025 ${base_height/2 + 0.005}" rpy="0 0 -${3.14/6}" />
+        <origin xyz="0.025 0.025 ${base_height/2 + 0.005}" rpy="0 0  1.57" />
     </xacro:range_sensor>
     <xacro:range_sensor name="range_sensor_left" parent="base_link">
-        <origin xyz="0.025 -0.025 ${base_height/2 + 0.005}" rpy="0 0 ${3.14/6}" />
+        <origin xyz="0.025 -0.025 ${base_height/2 + 0.005}" rpy="0 0 -1.57" />
     </xacro:range_sensor>
-    <xacro:range_sensor name="range_sensor_front" parent="base_link">
-        <origin xyz="0.025 0.0 ${base_height/2 + 0.005}" rpy="0 0 0" />
+    <xacro:range_sensor name="range_sensor_front_left" parent="base_link">
+        <origin xyz="0.025 -0.01 ${base_height/2 + 0.005}" rpy="0 0 0" />
+    </xacro:range_sensor>
+    <xacro:range_sensor name="range_sensor_front_right" parent="base_link">
+        <origin xyz="0.025 0.01 ${base_height/2 + 0.005}" rpy="0 0 0" />
     </xacro:range_sensor>
 </robot>

Commit message: Randomly driving maze

File: ws/src/micromouse_description/urdf/micromouse_description.xacro (robot description, xacro)
@@ -100,8 +100,8 @@
     <xacro:include filename="$(find micromouse_description)/urdf/range_sensor.xacro" />
     <xacro:range_sensor name="range_sensor_right" parent="base_link">
-        <origin xyz="0.025 0.025 ${base_height/2 + 0.005}" rpy="0 0  1.57" />
+        <origin xyz="0.025 0.025 ${base_height/2 + 0.005}" rpy="0 0  1.2" />
     </xacro:range_sensor>
     <xacro:range_sensor name="range_sensor_left" parent="base_link">
-        <origin xyz="0.025 -0.025 ${base_height/2 + 0.005}" rpy="0 0 -1.57" />
+        <origin xyz="0.025 -0.025 ${base_height/2 + 0.005}" rpy="0 0 -1.2" />
     </xacro:range_sensor>
     <xacro:range_sensor name="range_sensor_front_left" parent="base_link">
